Commit message: Fix swerve drive for navigation task and add curriculum learning for reach task.

File: source/robotis_sh5/data/robots/ffw_sh5_follower_copy.urdf (robot description, URDF)
Before this commit: robot ffw_sh5_follower, 90 links, 89 joints
Links:
- link arm_base_link: geometry collision mesh filename=package://ffw_description/meshes/common/follower/body_arm_a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 scale=0.001 0.001 0.001; visual mesh filename=package://ffw_description/meshes/common/follower/body_arm_a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 scale=0.001 0.001 0.001
- link arm_l_link1: geometry collision mesh filename=package://ffw_description/meshes/common/follower/arm_l_link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 scale=0.001 0.001 0.001; visual mesh filename=package://ffw_description/meshes/common/follower/arm_l_link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 scale=0.001 0.001 0.001
- link arm_l_link2: geometry collision mesh filename=package://ffw_description/meshes/common/follower/arm_l_link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 scale=0.001 0.001 0.001; visual mesh filename=package://ffw_description/meshes/common/follower/arm_l_link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 scale=0.001 0.001 0.001
- link arm_l_link3: geometry collision mesh filename=package://ffw_description/meshes/common/follower/arm_l_link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 scale=0.001 0.001 0.001; visual mesh filename=package://ffw_description/meshes/common/follower/arm_l_link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 scale=0.001 0.001 0.001
- link arm_l_link4: geometry collision mesh filename=package://ffw_description/meshes/common/follower/arm_l_link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 scale=0.001 0.001 0.001; visual mesh filename=package://ffw_description/meshes/common/follower/arm_l_link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 scale=0.001 0.001 0.001
- link arm_l_link5: geometry collision mesh filename=package://ffw_description/meshes/common/follower/arm_l_link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 scale=0.001 0.001 0.001; visual mesh filename=package://ffw_description/meshes/common/follower/arm_l_link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 scale=0.001 0.001 0.001
- link arm_l_link6: geometry collision mesh filename=package://ffw_description/meshes/common/follower/arm_l_link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 scale=0.001 0.001 0.001; visual mesh filename=package://ffw_description/meshes/common/follower/arm_l_link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 scale=0.001 0.001 0.001
- link arm_l_link7: geometry collision mesh filename=package://ffw_description/meshes/common/follower/arm_l_link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 scale=0.001 0.001 0.001; visual mesh filename=package://ffw_description/meshes/common/follower/arm_l_link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 scale=0.001 0.001 0.001
- link arm_r_link1: geometry collision mesh filename=package://ffw_description/meshes/common/follower/arm_r_link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 scale=0.001 0.001 0.001; visual mesh filename=package://ffw_description/meshes/common/follower/arm_r_link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 scale=0.001 0.001 0.001
- link arm_r_link2: geometry collision mesh filename=package://ffw_description/meshes/common/follower/arm_r_link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 scale=0.001 0.001 0.001; visual mesh filename=package://ffw_description/meshes/common/follower/arm_r_link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 scale=0.001 0.001 0.001
- link arm_r_link3: geometry collision mesh filename=package://ffw_description/meshes/common/follower/arm_r_link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 scale=0.001 0.001 0.001; visual mesh filename=package://ffw_description/meshes/common/follower/arm_r_link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 scale=0.001 0.001 0.001
- link arm_r_link4: geometry collision mesh filename=package://ffw_description/meshes/common/follower/arm_r_link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 scale=0.001 0.001 0.001; visual mesh filename=package://ffw_description/meshes/common/follower/arm_r_link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 scale=0.001 0.001 0.001
- link arm_r_link5: geometry collision mesh filename=package://ffw_description/meshes/common/follower/arm_r_link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 scale=0.001 0.001 0.001; visual mesh filename=package://ffw_description/meshes/common/follower/arm_r_link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 scale=0.001 0.001 0.001
- link arm_r_link6: geometry collision mesh filename=package://ffw_description/meshes/common/follower/arm_r_link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 scale=0.001 0.001 0.001; visual mesh filename=package://ffw_description/meshes/common/follower/arm_r_link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 scale=0.001 0.001 0.001
- link arm_r_link7: geometry collision mesh filename=package://ffw_description/meshes/common/follower/arm_r_link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 scale=0.001 0.001 0.001; visual mesh filename=package://ffw_description/meshes/common/follower/arm_r_link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 scale=0.001 0.001 0.001
- link camera_l_link: geometry collision box size=0.023 0.042 0.042; visual mesh filename=file:///root/ros2_ws/install/realsense2_description/share/r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 scale=0.001 0.001 0.001
- link camera_r_link: geometry collision box size=0.023 0.042 0.042; visual mesh filename=file:///root/ros2_ws/install/realsense2_description/share/r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 scale=0.001 0.001 0.001
- link finger_l_link1: geometry collision mesh filename=package://ffw_description/meshes/common/hx5_d20/hx5_d20_lef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 scale=0.001 0.001 0.001; visual mesh filename=package://ffw_description/meshes/common/hx5_d20/hx5_d20_lef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 scale=0.001 0.001 0.001
- link finger_l_link10: geometry collision mesh filename=package://ffw_description/meshes/common/hx5_d20/hx5_d20_lef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 scale=0.001 0.001 0.001; visual mesh filename=package://ffw_description/meshes/common/hx5_d20/hx5_d20_lef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 scale=0.001 0.001 0.001
- link finger_l_link11: geometry collision mesh filename=package://ffw_description/meshes/common/hx5_d20/hx5_d20_lef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 scale=0.001 0.001 0.001; visual mesh filename=package://ffw_description/meshes/common/hx5_d20/hx5_d20_lef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 scale=0.001 0.001 0.001
- link finger_l_link12: geometry collision mesh filename=package://ffw_description/meshes/common/hx5_d20/hx5_d20_lef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 scale=0.001 0.001 0.001; visual mesh filename=package://ffw_description/meshes/common/hx5_d20/hx5_d20_lef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 scale=0.001 0.001 0.001
- link finger_l_link13: geometry collision mesh filename=package://ffw_description/meshes/common/hx5_d20/hx5_d20_lef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 scale=0.001 0.001 0.001; visual mesh filename=package://ffw_description/meshes/common/hx5_d20/hx5_d20_lef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 scale=0.001 0.001 0.001
- link finger_l_link14: geometry collision mesh filename=package://ffw_description/meshes/common/hx5_d20/hx5_d20_lef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 scale=0.001 0.001 0.001; visual mesh filename=package://ffw_description/meshes/common/hx5_d20/hx5_d20_lef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 scale=0.001 0.001 0.001
- link finger_l_link15: geometry collision mesh filename=package://ffw_description/meshes/common/hx5_d20/hx5_d20_lef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 scale=0.001 0.001 0.001; visual mesh filename=package://ffw_description/meshes/common/hx5_d20/hx5_d20_lef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 scale=0.001 0.001 0.001
- link finger_l_link16: geometry collision mesh filename=package://ffw_description/meshes/common/hx5_d20/hx5_d20_lef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 scale=0.001 0.001 0.001; visual mesh filename=package://ffw_description/meshes/common/hx5_d20/hx5_d20_lef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 scale=0.001 0.001 0.001
- link finger_l_link17: geometry collision mesh filename=package://ffw_description/meshes/common/hx5_d20/hx5_d20_lef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 scale=0.001 0.001 0.001; visual mesh filename=package://ffw_description/meshes/common/hx5_d20/hx5_d20_lef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 scale=0.001 0.001 0.001
- link finger_l_link18: geometry collision mesh filename=package://ffw_description/meshes/common/hx5_d20/hx5_d20_lef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 scale=0.001 0.001 0.001; visual mesh filename=package://ffw_description/meshes/common/hx5_d20/hx5_d20_lef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 scale=0.001 0.001 0.001
- link finger_l_link19: geometry collision mesh filename=package://ffw_description/meshes/common/hx5_d20/hx5_d20_lef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 scale=0.001 0.001 0.001; visual mesh filename=package://ffw_description/meshes/common/hx5_d20/hx5_d20_lef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 scale=0.001 0.001 0.001
- link finger_l_link2: geometry collision mesh filename=package://ffw_description/meshes/common/hx5_d20/hx5_d20_lef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 scale=0.001 0.001 0.001; visual mesh filename=package://ffw_description/meshes/common/hx5_d20/hx5_d20_lef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 scale=0.001 0.001 0.001
- link finger_l_link20: geometry collision mesh filename=package://ffw_description/meshes/common/hx5_d20/hx5_d20_lef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 scale=0.001 0.001 0.001; visual mesh filename=package://ffw_description/meshes/common/hx5_d20/hx5_d20_lef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 scale=0.001 0.001 0.001
- link finger_l_link3: geometry collision mesh filename=package://ffw_description/meshes/common/hx5_d20/hx5_d20_lef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 scale=0.001 0.001 0.001; visual mesh filename=package://ffw_description/meshes/common/hx5_d20/hx5_d20_lef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 scale=0.001 0.001 0.001
- link finger_l_link4: geometry collision mesh filename=package://ffw_description/meshes/common/hx5_d20/hx5_d20_lef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 scale=0.001 0.001 0.001; visual mesh filename=package://ffw_description/meshes/common/hx5_d20/hx5_d20_lef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 scale=0.001 0.001 0.001
- link finger_l_link5: geometry collision mesh filename=package://ffw_description/meshes/common/hx5_d20/hx5_d20_lef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 scale=0.001 0.001 0.001; visual mesh filename=package://ffw_description/meshes/common/hx5_d20/hx5_d20_lef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 scale=0.001 0.001 0.001
- link finger_l_link6: geometry collision mesh filename=package://ffw_description/meshes/common/hx5_d20/hx5_d20_lef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 scale=0.001 0.001 0.001; visual mesh filename=package://ffw_description/meshes/common/hx5_d20/hx5_d20_lef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 scale=0.001 0.001 0.001
- link finger_l_link7: geometry collision mesh filename=package://ffw_description/meshes/common/hx5_d20/hx5_d20_lef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 scale=0.001 0.001 0.001; visual mesh filename=package://ffw_description/meshes/common/hx5_d20/hx5_d20_lef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 scale=0.001 0.001 0.001
- link finger_l_link8: geometry collision mesh filename=package://ffw_description/meshes/common/hx5_d20/hx5_d20_lef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 scale=0.001 0.001 0.001; visual mesh filename=package://ffw_description/meshes/common/hx5_d20/hx5_d20_lef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 scale=0.001 0.001 0.001
- link finger_l_link9: geometry collision mesh filename=package://ffw_description/meshes/common/hx5_d20/hx5_d20_lef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 scale=0.001 0.001 0.001; visual mesh filename=package://ffw_description/meshes/common/hx5_d20/hx5_d20_lef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 scale=0.001 0.001 0.001
- link finger_r_link1: geometry collision mesh filename=package://ffw_description/meshes/common/hx5_d20/hx5_d20_rig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 scale=0.001 0.001 0.001; visual mesh filename=package://ffw_description/meshes/common/hx5_d20/hx5_d20_rig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 scale=0.001 0.001 0.001
- link finger_r_link10: geometry collision mesh filename=package://ffw_description/meshes/common/hx5_d20/hx5_d20_rig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 scale=0.001 0.001 0.001; visual mesh filename=package://ffw_description/meshes/common/hx5_d20/hx5_d20_rig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 scale=0.001 0.001 0.001
- link finger_r_link11: geometry collision mesh filename=package://ffw_description/meshes/common/hx5_d20/hx5_d20_rig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 scale=0.001 0.001 0.001; visual mesh filename=package://ffw_description/meshes/common/hx5_d20/hx5_d20_rig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 scale=0.001 0.001 0.001
- link finger_r_link12: geometry collision mesh filename=package://ffw_description/meshes/common/hx5_d20/hx5_d20_rig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 scale=0.001 0.001 0.001; visual mesh filename=package://ffw_description/meshes/common/hx5_d20/hx5_d20_rig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 scale=0.001 0.001 0.001
- link finger_r_link13: geometry collision mesh filename=package://ffw_description/meshes/common/hx5_d20/hx5_d20_rig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 scale=0.001 0.001 0.001; visual mesh filename=package://ffw_description/meshes/common/hx5_d20/hx5_d20_rig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 scale=0.001 0.001 0.001
- link finger_r_link14: geometry collision mesh filename=package://ffw_description/meshes/common/hx5_d20/hx5_d20_rig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 scale=0.001 0.001 0.001; visual mesh filename=package://ffw_description/meshes/common/hx5_d20/hx5_d20_rig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 scale=0.001 0.001 0.001
- link finger_r_link15: geometry collision mesh filename=package://ffw_description/meshes/common/hx5_d20/hx5_d20_rig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 scale=0.001 0.001 0.001; visual mesh filename=package://ffw_description/meshes/common/hx5_d20/hx5_d20_rig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 scale=0.001 0.001 0.001
- link finger_r_link16: geometry collision mesh filename=package://ffw_description/meshes/common/hx5_d20/hx5_d20_rig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 scale=0.001 0.001 0.001; visual mesh filename=package://ffw_description/meshes/common/hx5_d20/hx5_d20_rig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 scale=0.001 0.001 0.001
- link finger_r_link17: geometry collision mesh filename=package://ffw_description/meshes/common/hx5_d20/hx5_d20_rig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 scale=0.001 0.001 0.001; visual mesh filename=package://ffw_description/meshes/common/hx5_d20/hx5_d20_rig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 scale=0.001 0.001 0.001
- link finger_r_link18: geometry collision mesh filename=package://ffw_description/meshes/common/hx5_d20/hx5_d20_rig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 scale=0.001 0.001 0.001; visual mesh filename=package://ffw_description/meshes/common/hx5_d20/hx5_d20_rig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 scale=0.001 0.001 0.001
- link finger_r_link19: geometry collision mesh filename=package://ffw_description/meshes/common/hx5_d20/hx5_d20_rig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 scale=0.001 0.001 0.001; visual mesh filename=package://ffw_description/meshes/common/hx5_d20/hx5_d20_rig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 scale=0.001 0.001 0.001
- link finger_r_link2: geometry collision mesh filename=package://ffw_description/meshes/common/hx5_d20/hx5_d20_rig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 scale=0.001 0.001 0.001; visual mesh filename=package://ffw_description/meshes/common/hx5_d20/hx5_d20_rig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 scale=0.001 0.001 0.001
- link finger_r_link20: geometry collision mesh filename=package://ffw_description/meshes/common/hx5_d20/hx5_d20_rig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 scale=0.001 0.001 0.001; visual mesh filename=package://ffw_description/meshes/common/hx5_d20/hx5_d20_rig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 scale=0.001 0.001 0.001
- link finger_r_link3: geometry collision mesh filename=package://ffw_description/meshes/common/hx5_d20/hx5_d20_rig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 scale=0.001 0.001 0.001; visual mesh filename=package://ffw_description/meshes/common/hx5_d20/hx5_d20_rig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 scale=0.001 0.001 0.001
- link finger_r_link4: geometry collision mesh filename=package://ffw_description/meshes/common/hx5_d20/hx5_d20_rig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 scale=0.001 0.001 0.001; visual mesh filename=package://ffw_description/meshes/common/hx5_d20/hx5_d20_rig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 scale=0.001 0.001 0.001
- link finger_r_link5: geometry collision mesh filename=package://ffw_description/meshes/common/hx5_d20/hx5_d20_rig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 scale=0.001 0.001 0.001; visual mesh filename=package://ffw_description/meshes/common/hx5_d20/hx5_d20_rig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 scale=0.001 0.001 0.001
- link finger_r_link6: geometry collision mesh filename=package://ffw_description/meshes/common/hx5_d20/hx5_d20_rig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 scale=0.001 0.001 0.001; visual mesh filename=package://ffw_description/meshes/common/hx5_d20/hx5_d20_rig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 scale=0.001 0.001 0.001
- link finger_r_link7: geometry collision mesh filename=package://ffw_description/meshes/common/hx5_d20/hx5_d20_rig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 scale=0.001 0.001 0.001; visual mesh filename=package://ffw_description/meshes/common/hx5_d20/hx5_d20_rig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 scale=0.001 0.001 0.001
- link finger_r_link8: geometry collision mesh filename=package://ffw_description/meshes/common/hx5_d20/hx5_d20_rig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 scale=0.001 0.001 0.001; visual mesh filename=package://ffw_description/meshes/common/hx5_d20/hx5_d20_rig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 scale=0.001 0.001 0.001
- link finger_r_link9: geometry collision mesh filename=package://ffw_description/meshes/common/hx5_d20/hx5_d20_rig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 scale=0.001 0.001 0.001; visual mesh filename=package://ffw_description/meshes/common/hx5_d20/hx5_d20_rig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 scale=0.001 0.001 0.001
- link head_link1: geometry collision mesh filename=package://ffw_description/meshes/common/follower/head_link1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 scale=0.001 0.001 0.001; visual mesh filename=package://ffw_description/meshes/common/follower/head_link1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 scale=0.001 0.001 0.001
- link head_link2: geometry collision mesh filename=package://ffw_description/meshes/common/follower/head_link2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 scale=0.001 0.001 0.001; visual mesh filename=package://ffw_description/meshes/common/follower/head_link2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 scale=0.001 0.001 0.001
- link hx5_d20_left_base: geometry collision mesh filename=package://ffw_description/meshes/common/hx5_d20/hx5_d20_lef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 scale=0.001 0.001 0.001; visual mesh filename=package://ffw_description/meshes/common/hx5_d20/hx5_d20_lef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 scale=0.001 0.001 0.001
- link hx5_d20_right_base: geometry collision mesh filename=package://ffw_description/meshes/common/hx5_d20/hx5_d20_rig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 scale=0.001 0.001 0.001; visual mesh filename=package://ffw_description/meshes/common/hx5_d20/hx5_d20_rig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 scale=0.001 0.001 0.001
- link left_wheel_drive_link: geometry collision cylinder length=0.05 radius=0.0865; visual mesh filename=../../meshes/ffw_sh5_rev1_follower/left_wheel_drive_link.stl scale=0.001 0.001 0.001
- link lift_link: mass 1.790000000e+01 -> 17.9
- link rear_wheel_drive_link: geometry collision cylinder length=0.05 radius=0.0865; visual mesh filename=../../meshes/ffw_sh5_rev1_follower/rear_wheel_drive_link.stl scale=0.001 0.001 0.001
- link right_wheel_drive_link: geometry collision cylinder length=0.05 radius=0.0865; visual mesh filename=../../meshes/ffw_sh5_rev1_follower/right_wheel_drive_link.s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 scale=0.001 0.001 0.001
- link zedm_camera_center: geometry collision mesh filename=file:///root/ros2_ws/install/ffw_description/share/ffw_desc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 scale=0.001 0.001 0.001; visual mesh filename=file:///root/ros2_ws/install/ffw_description/share/ffw_desc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 scale=0.001 0.001 0.001
